Commit message: import two robots model, and fix urdf file for robot model (whole robot)

File: Assets/Urdf/ai_robot/robot_ai.urdf (robot description, URDF)
Before this commit: robot ai_robot, 1 links, 0 joints
Links:
- link base_link: geometry collision box size=0.2 0.12 0.26; collision box size=0.569 0.452 0.14
